File: Carrier-Board.kicad_pcb (KiCad board)
At the start: 2 copper layers, 0 parts

Commit message: Add converted PC104-plus connector from eagle libs
Parts:
- added X1: PC104_PLUS, Carrier-Board:con-pc104-PC104-PLUS, F.Cu at (56.5, 127.0)
