File: Carrier-Board.kicad_pcb (KiCad board)
At the start: 2 copper layers, 92 x 96 mm, 39 parts, among them J1 CONN_3-6318491-6, J3 Conn_02x26_Odd_Even, J4 SI-51009-F, J5 Conn_02x26_Odd_Even, J6 Conn_01x03_Male, J7 Conn_01x03_Male, J8 Conn_01x06_Male, U1 MPM3620, U2 MPM3620, U9 MSATA-Socket

Commit message: schematic 90% done
Parts:
- added J9: Conn_02x04_Odd_Even, Pin_Headers:Pin_Header_Angled_2x04_Pitch2.54mm, F.Cu at (265.9, 149.7)
Changed lines of the file:
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@@
     (tracks 0)
     (zones 0)
-    (modules 39)
-    (nets 352)
+    (modules 40)
+    (nets 360)
   )
   (page A4)
@@
   (net 350 "Net-(J3-Pad51)")
   (net 351 "Net-(J3-Pad52)")
+  (net 352 "Net-(J9-Pad1)")
+  (net 353 "Net-(J9-Pad2)")
+  (net 354 "Net-(J9-Pad3)")
+  (net 355 "Net-(J9-Pad4)")
+  (net 356 "Net-(J9-Pad5)")
+  (net 357 "Net-(J9-Pad6)")
+  (net 358 "Net-(J9-Pad7)")
+  (net 359 "Net-(J9-Pad8)")
   (net_class Default "This is the default net class."
     (clearance 0.2)
@@
     (add_net "Net-(J5-Pad8)")
     (add_net "Net-(J5-Pad9)")
+    (add_net "Net-(J9-Pad1)")
+    (add_net "Net-(J9-Pad2)")
+    (add_net "Net-(J9-Pad3)")
+    (add_net "Net-(J9-Pad4)")
+    (add_net "Net-(J9-Pad5)")
+    (add_net "Net-(J9-Pad6)")
+    (add_net "Net-(J9-Pad7)")
+    (add_net "Net-(J9-Pad8)")
     (add_net "Net-(R1-Pad2)")
     (add_net "Net-(R3-Pad2)")
@@
       (at (xyz 0 0 0))
       (scale (xyz 1 1 1))
+      (rotate (xyz 0 0 0))
+    )
+  )
+  (module Pin_Headers:Pin_Header_Angled_2x04_Pitch2.54mm (layer F.Cu)
+    (at 265.925 149.725)
+    (descr "Through hole angled pin header, 2x04, 2.54mm pitch, 6mm pin length, double rows")
+    (tags "Through hole angled pin header THT 2x04 2.54mm double row")
+    (fp_text reference J9 (at 5.655 -2.27) (layer F.SilkS)
+      (effects (font (size 1 1) (thickness 0.15)))
+    )
+    (fp_text value Conn_02x04_Odd_Even (at 5.655 9.89) (layer F.Fab)
+      (effects (font (size 1 1) (thickness 0.15)))
+    )
+    (fp_line (start 4.675 -1.27) (end 6.58 -1.27) (layer F.Fab) (width 0.1))
+    (fp_line (start 6.58 -1.27) (end 6.58 8.89) (layer F.Fab) (width 0.1))
+    (fp_line (start 6.58 8.89) (end 4.04 8.89) (layer F.Fab) (width 0.1))
+    (fp_line (start 4.04 8.89) (end 4.04 -0.635) (layer F.Fab) (width 0.1))
+    (fp_line (start 4.04 -0.635) (end 4.675 -1.27) (layer F.Fab) (width 0.1))
+    (fp_line (start -0.32 -0.32) (end 4.04 -0.32) (layer F.Fab) (width 0.1))
+    (fp_line (start -0.32 -0.32) (end -0.32 0.32) (layer F.Fab) (width 0.1))
+    (fp_line (start -0.32 0.32) (end 4.04 0.32) (layer F.Fab) (width 0.1))
+    (fp_line (start 6.58 -0.32) (end 12.58 -0.32) (layer F.Fab) (width 0.1))
+    (fp_line (start 12.58 -0.32) (end 12.58 0.32) (layer F.Fab) (width 0.1))
+    (fp_line (start 6.58 0.32) (end 12.58 0.32) (layer F.Fab) (width 0.1))
+    (fp_line (start -0.32 2.22) (end 4.04 2.22) (layer F.Fab) (width 0.1))
+    (fp_line (start -0.32 2.22) (end -0.32 2.86) (layer F.Fab) (width 0.1))
+    (fp_line (start -0.32 2.86) (end 4.04 2.86) (layer F.Fab) (width 0.1))
+    (fp_line (start 6.58 2.22) (end 12.58 2.22) (layer F.Fab) (width 0.1))
+    (fp_line (start 12.58 2.22) (end 12.58 2.86) (layer F.Fab) (width 0.1))
+    (fp_line (start 6.58 2.86) (end 12.58 2.86) (layer F.Fab) (width 0.1))
+    (fp_line (start -0.32 4.76) (end 4.04 4.76) (layer F.Fab) (width 0.1))
+    (fp_line (start -0.32 4.76) (end -0.32 5.4) (layer F.Fab) (width 0.1))
+    (fp_line (start -0.32 5.4) (end 4.04 5.4) (layer F.Fab) (width 0.1))
+    (fp_line (start 6.58 4.76) (end 12.58 4.76) (layer F.Fab) (width 0.1))
+    (fp_line (start 12.58 4.76) (end 12.58 5.4) (layer F.Fab) (width 0.1))
+    (fp_line (start 6.58 5.4) (end 12.58 5.4) (layer F.Fab) (width 0.1))
+    (fp_line (start -0.32 7.3) (end 4.04 7.3) (layer F.Fab) (width 0.1))
+    (fp_line (start -0.32 7.3) (end -0.32 7.94) (layer F.Fab) (width 0.1))
+    (fp_line (start -0.32 7.94) (end 4.04 7.94) (layer F.Fab) (width 0.1))
+    (fp_line (start 6.58 7.3) (end 12.58 7.3) (layer F.Fab) (width 0.1))
+    (fp_line (start 12.58 7.3) (end 12.58 7.94) (layer F.Fab) (width 0.1))
+    (fp_line (start 6.58 7.94) (end 12.58 7.94) (layer F.Fab) (width 0.1))
+    (fp_line (start 3.98 -1.33) (end 3.98 8.95) (layer F.SilkS) (width 0.12))
+    (fp_line (start 3.98 8.95) (end 6.64 8.95) (layer F.SilkS) (width 0.12))
+    (fp_line (start 6.64 8.95) (end 6.64 -1.33) (layer F.SilkS) (width 0.12))
+    (fp_line (start 6.64 -1.33) (end 3.98 -1.33) (layer F.SilkS) (width 0.12))
+    (fp_line (start 6.64 -0.38) (end 12.64 -0.38) (layer F.SilkS) (width 0.12))
+    (fp_line (start 12.64 -0.38) (end 12.64 0.38) (layer F.SilkS) (width 0.12))
+    (fp_line (start 12.64 0.38) (end 6.64 0.38) (layer F.SilkS) (width 0.12))
+    (fp_line (start 6.64 -0.32) (end 12.64 -0.32) (layer F.SilkS) (width 0.12))
+    (fp_line (start 6.64 -0.2) (end 12.64 -0.2) (layer F.SilkS) (width 0.12))
+    (fp_line (start 6.64 -0.08) (end 12.64 -0.08) (layer F.SilkS) (width 0.12))
+    (fp_line (start 6.64 0.04) (end 12.64 0.04) (layer F.SilkS) (width 0.12))
+    (fp_line (start 6.64 0.16) (end 12.64 0.16) (layer F.SilkS) (width 0.12))
+    (fp_line (start 6.64 0.28) (end 12.64 0.28) (layer F.SilkS) (width 0.12))
+    (fp_line (start 3.582929 -0.38) (end 3.98 -0.38) (layer F.SilkS) (width 0.12))
+    (fp_line (start 3.582929 0.38) (end 3.98 0.38) (layer F.SilkS) (width 0.12))
+    (fp_line (start 1.11 -0.38) (end 1.497071 -0.38) (layer F.SilkS) (width 0.12))
+    (fp_line (start 1.11 0.38) (end 1.497071 0.38) (layer F.SilkS) (width 0.12))
+    (fp_line (start 3.98 1.27) (end 6.64 1.27) (layer F.SilkS) (width 0.12))
+    (fp_line (start 6.64 2.16) (end 12.64 2.16) (layer F.SilkS) (width 0.12))
+    (fp_line (start 12.64 2.16) (end 12.64 2.92) (layer F.SilkS) (width 0.12))
+    (fp_line (start 12.64 2.92) (end 6.64 2.92) (layer F.SilkS) (width 0.12))
+    (fp_line (start 3.582929 2.16) (end 3.98 2.16) (layer F.SilkS) (width 0.12))
+    (fp_line (start 3.582929 2.92) (end 3.98 2.92) (layer F.SilkS) (width 0.12))
+    (fp_line (start 1.042929 2.16) (end 1.497071 2.16) (layer F.SilkS) (width 0.12))
+    (fp_line (start 1.042929 2.92) (end 1.497071 2.92) (layer F.SilkS) (width 0.12))
+    (fp_line (start 3.98 3.81) (end 6.64 3.81) (layer F.SilkS) (width 0.12))
+    (fp_line (start 6.64 4.7) (end 12.64 4.7) (layer F.SilkS) (width 0.12))
+    (fp_line (start 12.64 4.7) (end 12.64 5.46) (layer F.SilkS) (width 0.12))
+    (fp_line (start 12.64 5.46) (end 6.64 5.46) (layer F.SilkS) (width 0.12))
+    (fp_line (start 3.582929 4.7) (end 3.98 4.7) (layer F.SilkS) (width 0.12))
+    (fp_line (start 3.582929 5.46) (end 3.98 5.46) (layer F.SilkS) (width 0.12))
+    (fp_line (start 1.042929 4.7) (end 1.497071 4.7) (layer F.SilkS) (width 0.12))
+    (fp_line (start 1.042929 5.46) (end 1.497071 5.46) (layer F.SilkS) (width 0.12))
+    (fp_line (start 3.98 6.35) (end 6.64 6.35) (layer F.SilkS) (width 0.12))
+    (fp_line (start 6.64 7.24) (end 12.64 7.24) (layer F.SilkS) (width 0.12))
+    (fp_line (start 12.64 7.24) (end 12.64 8) (layer F.SilkS) (width 0.12))
+    (fp_line (start 12.64 8) (end 6.64 8) (layer F.SilkS) (width 0.12))
+    (fp_line (start 3.582929 7.24) (end 3.98 7.24) (layer F.SilkS) (width 0.12))
+    (fp_line (start 3.582929 8) (end 3.98 8) (layer F.SilkS) (width 0.12))
+    (fp_line (start 1.042929 7.24) (end 1.497071 7.24) (layer F.SilkS) (width 0.12))
+    (fp_line (start 1.042929 8) (end 1.497071 8) (layer F.SilkS) (width 0.12))
+    (fp_line (start -1.27 0) (end -1.27 -1.27) (layer F.SilkS) (width 0.12))
+    (fp_line (start -1.27 -1.27) (end 0 -1.27) (layer F.SilkS) (width 0.12))
+    (fp_line (start -1.8 -1.8) (end -1.8 9.4) (layer F.CrtYd) (width 0.05))
+    (fp_line (start -1.8 9.4) (end 13.1 9.4) (layer F.CrtYd) (width 0.05))
+    (fp_line (start 13.1 9.4) (end 13.1 -1.8) (layer F.CrtYd) (width 0.05))
+    (fp_line (start 13.1 -1.8) (end -1.8 -1.8) (layer F.CrtYd) (width 0.05))
+    (fp_text user %R (at 5.31 3.81 90) (layer F.Fab)
+      (effects (font (size 1 1) (thickness 0.15)))
+    )
+    (pad 1 thru_hole rect (at 0 0) (size 1.7 1.7) (drill 1) (layers *.Cu *.Mask)
+      (net 352 "Net-(J9-Pad1)"))
+    (pad 2 thru_hole oval (at 2.54 0) (size 1.7 1.7) (drill 1) (layers *.Cu *.Mask)
+      (net 353 "Net-(J9-Pad2)"))
+    (pad 3 thru_hole oval (at 0 2.54) (size 1.7 1.7) (drill 1) (layers *.Cu *.Mask)
+      (net 354 "Net-(J9-Pad3)"))
+    (pad 4 thru_hole oval (at 2.54 2.54) (size 1.7 1.7) (drill 1) (layers *.Cu *.Mask)
+      (net 355 "Net-(J9-Pad4)"))
+    (pad 5 thru_hole oval (at 0 5.08) (size 1.7 1.7) (drill 1) (layers *.Cu *.Mask)
+      (net 356 "Net-(J9-Pad5)"))
+    (pad 6 thru_hole oval (at 2.54 5.08) (size 1.7 1.7) (drill 1) (layers *.Cu *.Mask)
+      (net 357 "Net-(J9-Pad6)"))
+    (pad 7 thru_hole oval (at 0 7.62) (size 1.7 1.7) (drill 1) (layers *.Cu *.Mask)
+      (net 358 "Net-(J9-Pad7)"))
+    (pad 8 thru_hole oval (at 2.54 7.62) (size 1.7 1.7) (drill 1) (layers *.Cu *.Mask)
+      (net 359 "Net-(J9-Pad8)"))
+    (model ${KISYS3DMOD}/Pin_Headers.3dshapes/Pin_Header_Angled_2x04_Pitch2.54mm.wrl
+      (at (xyz 0 0 0))
+      (scale (xyz 1 1 1))

Commit message: began layot
added dc jack, fixed ethernet footptrint aligned pc104
Parts:
- added J2: Conn_01x0, Connectors:Barrel_Jack_CUI_PJ-036AH-SMT, F.Cu at (90.0, 71.0)
- J1: value CONN_3-6318491-6 -> ComExpressMini
- U9: footprint BusSimulator:msata-socket -> Carrier-Board:mpcie-socket
- moved J4 185.9 mm to (76.5, 49.2)
- moved U9 160.6 mm to (92.9, 91.1)
- moved J1 154.0 mm to (165.7, 110.8)
- moved J8 150.1 mm to (168.8, 88.3)
- moved J9 144.3 mm to (166.7, 45.0)
- moved J6 122.0 mm to (169.2, 57.0)
- moved J7 99.0 mm to (168.8, 78.2)
- moved REF** 82.3 mm to (83.9, 120.0)
- moved G1 58.6 mm to (213.0, 78.0)
Connections:
- C1 pad 1: Net-(C1-Pad1) -> +12V
- C1 pad 2: Net-(C1-Pad2) -> mCOM_GND
- C2 pad 1: Net-(C2-Pad1) -> mCOM_5V_SBY
- C2 pad 2: Net-(C2-Pad2) -> mCOM_GND
- C3 pad 1: Net-(C3-Pad1) -> mCOM_GND
- C3 pad 2: Net-(C3-Pad2) -> +12V
- C4 pad 1: Net-(C4-Pad1) -> +3.3V
- C4 pad 2: Net-(C4-Pad2) -> mCOM_GND
- D5 pad 1: 12v_sense -> mCOM_12V
- J1 pad 104: 12v_sense -> mCOM_12V
- J1 pad 105: 12v_sense -> mCOM_12V
- J1 pad 106: 12v_sense -> mCOM_12V
- J1 pad 107: 12v_sense -> mCOM_12V
- J1 pad 108: 12v_sense -> mCOM_12V
- J1 pad 109: 12v_sense -> mCOM_12V
- J1 pad 214: 12v_sense -> mCOM_12V
- J1 pad 215: 12v_sense -> mCOM_12V
- J1 pad 216: 12v_sense -> mCOM_12V
- J1 pad 217: 12v_sense -> mCOM_12V
- J1 pad 218: 12v_sense -> mCOM_12V
- J1 pad 219: 12v_sense -> mCOM_12V
- R3 pad 1: 12v_sense -> +12V
- R7 pad 1: 12v_sense -> +12V
- U1 pad 16: 12v_sense -> +12V
- U2 pad 16: 12v_sense -> +12V

Commit message: Finished Schmatic
Didnt do pc104 connector
Parts:
- removed R10, R12, R9: 10k, Resistors_SMD:R_0603
- removed R11: 30k, Resistors_SMD:R_0603
- D5, R23, R24, R25: moved to B.Cu
- J1: value ComExpressMini -> CONN_3-6318491-6
- moved R23 246.4 mm to (86.2, 111.6)
- moved D8 220.0 mm to (87.0, 101.8)
- moved D5 219.2 mm to (91.5, 105.8)
- moved R2 206.3 mm to (109.2, 108.0)
- moved D6 205.5 mm to (87.0, 111.0)
- moved C2 202.6 mm to (114.8, 100.5), turned to 90 degrees
- moved R6 201.5 mm to (132.6, 104.5)
- moved R4 196.2 mm to (110.2, 98.8)
- moved R24 193.2 mm to (86.2, 106.3)
- moved C1 191.2 mm to (118.5, 108.2)
- moved C3 175.5 mm to (135.2, 108.5)
- moved R25 172.2 mm to (86.2, 101.1)
- moved D7 171.3 mm to (87.0, 106.2)
- moved R3 171.2 mm to (112.5, 108.2)
- moved R32 169.1 mm to (161.1, 66.0)
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Connections:
- C3 pad 1: mCOM_GND -> +12V
- C3 pad 2: +12V -> mCOM_GND

Commit message: added buttons
Parts:
- added J10: Conn_02x03_Odd_Even, Pin_Headers:Pin_Header_Angled_2x03_Pitch2.54mm, F.Cu at (88.8, 107.0)
- added R9: 330, Resistors_SMD:R_0805, F.Cu at (104.0, 79.5)
- added SW1: SW_Push, Buttons_Switches_SMD:SW_SPST_PTS645, F.Cu at (87.7, 41.0)
- added SW2: SW_Push, Buttons_Switches_SMD:SW_SPST_PTS645, F.Cu at (98.8, 59.0)
- added SW3: SW_Push, Buttons_Switches_SMD:SW_SPST_PTS645, F.Cu at (99.7, 70.5)
- C1, C2, C3, C4, R1, R2, R3, R4, R5, R6, R7, R8, U1, U2: moved to B.Cu
- moved R23 34.5 mm to (117.6, 97.3), turned to 90 degrees
- moved D6 32.4 mm to (116.5, 97.5), turned to 90 degrees
- moved R24 27.6 mm to (112.3, 97.3), turned to 90 degrees
- moved D7 26.3 mm to (111.8, 97.5), turned to 90 degrees
- moved D5 24.5 mm to (111.8, 92.0), turned to 90 degrees
- moved R25 21.2 mm to (107.1, 97.3), turned to 90 degrees
- moved D8 20.7 mm to (107.2, 97.5), turned to 90 degrees
- moved R4 13.8 mm to (113.2, 112.2)
- moved C4 13.3 mm to (136.2, 112.0), turned to 270 degrees
- moved C2 10.4 mm to (117.8, 110.5), turned to 270 degrees
- moved J7 8.50 mm to (87.8, 73.8)
- moved J8 8.50 mm to (87.8, 63.8)
- moved C3 6.75 mm to (138.2, 102.5)
- moved R7 6.30 mm to (128.3, 102.7)
- moved C1 6.30 mm to (121.5, 102.7)
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Connections:
- C1 pad 1: +12V -> mCOM_12V
- C1 pad 2: mCOM_GND -> GBE0_CTREF(GND)
- C2 pad 2: mCOM_GND -> GBE0_CTREF(GND)
- C27 pad 2: mCOM_GND -> GBE0_CTREF(GND)
- C28 pad 2: mCOM_GND -> GBE0_CTREF(GND)
- C29 pad 2: mCOM_GND -> GBE0_CTREF(GND)
- C3 pad 1: +12V -> mCOM_12V
- C3 pad 2: mCOM_GND -> GBE0_CTREF(GND)
- C4 pad 2: mCOM_GND -> GBE0_CTREF(GND)
- J1 pad 1: mCOM_GND -> GBE0_CTREF(GND)
- J1 pad 10: Net-(J1-Pad10) -> GBE0_MDI1+
- J1 pad 100: mCOM_GND -> GBE0_CTREF(GND)
- J1 pad 11: mCOM_GND -> GBE0_CTREF(GND)
- J1 pad 110: mCOM_GND -> GBE0_CTREF(GND)
- J1 pad 111: mCOM_GND -> GBE0_CTREF(GND)
- J1 pad 12: Net-(J1-Pad12) -> GBE0_MDI0-
- J1 pad 121: mCOM_GND -> GBE0_CTREF(GND)
- J1 pad 13: Net-(J1-Pad13) -> GBE0_MDI0+
- J1 pad 131: mCOM_GND -> GBE0_CTREF(GND)
- J1 pad 14: Net-(J1-Pad14) -> GBE0_CTREF(GND)
- J1 pad 141: mCOM_GND -> GBE0_CTREF(GND)
- J1 pad 151: mCOM_GND -> GBE0_CTREF(GND)
- J1 pad 161: mCOM_GND -> GBE0_CTREF(GND)
- J1 pad 170: mCOM_GND -> GBE0_CTREF(GND)
- J1 pad 180: mCOM_GND -> GBE0_CTREF(GND)
- J1 pad 190: mCOM_GND -> GBE0_CTREF(GND)
- J1 pad 2: Net-(J1-Pad2) -> GBE0_MDI3-
- J1 pad 200: mCOM_GND -> GBE0_CTREF(GND)
- J1 pad 21: mCOM_GND -> GBE0_CTREF(GND)
- J1 pad 210: mCOM_GND -> GBE0_CTREF(GND)
- J1 pad 220: mCOM_GND -> GBE0_CTREF(GND)
- J1 pad 3: Net-(J1-Pad3) -> GBE0_MDI3+
- J1 pad 31: mCOM_GND -> GBE0_CTREF(GND)
- J1 pad 4: Net-(J1-Pad4) -> GBE0_LINK100#
- J1 pad 41: mCOM_GND -> GBE0_CTREF(GND)
- J1 pad 5: Net-(J1-Pad5) -> GBE0_LINK1000#
- J1 pad 51: mCOM_GND -> GBE0_CTREF(GND)
- J1 pad 57: mCOM_GND -> GBE0_CTREF(GND)
- J1 pad 6: Net-(J1-Pad6) -> GBE0_MDI2-
- J1 pad 60: mCOM_GND -> GBE0_CTREF(GND)
- J1 pad 66: mCOM_GND -> GBE0_CTREF(GND)
- J1 pad 7: Net-(J1-Pad7) -> GBE0_MDI2+
- J1 pad 70: mCOM_GND -> GBE0_CTREF(GND)
- J1 pad 80: mCOM_GND -> GBE0_CTREF(GND)
- J1 pad 9: Net-(J1-Pad9) -> GBE0_MDI1-
- J1 pad 90: mCOM_GND -> GBE0_CTREF(GND)
- J1 pad 92: Net-(J1-Pad92) -> SPI_MISO
- J1 pad 94: Net-(J1-Pad94) -> SPI_CLK
- J1 pad 95: Net-(J1-Pad95) -> SPI_MOSI
- J1 pad 97: Net-(J1-Pad97) -> SPI_CS#
- J2 pad 1: +12V -> mCOM_12V
- J2 pad 2: mCOM_GND -> GBE0_CTREF(GND)
- J2 pad 3: mCOM_GND -> GBE0_CTREF(GND)
- J4 pad 1: Net-(J4-Pad1) -> GBE0_CTREF(GND)
- J4 pad 10: Net-(J4-Pad10) -> GBE0_MDI3-
- J4 pad 13: (no net) -> GBE0_LINK1000#
- J4 pad 14: (no net) -> Net-(J4-Pad14)
- J4 pad 15: (no net) -> Net-(J4-Pad15)
- J4 pad 16: (no net) -> GBE0_LINK100#
- J4 pad 17: (no net) -> GBE0_CTREF(GND)
- J4 pad 18: (no net) -> GBE0_CTREF(GND)
- J4 pad 2: Net-(J4-Pad2) -> GBE0_MDI0+
- J4 pad 3: Net-(J4-Pad3) -> GBE0_MDI0-
- J4 pad 4: Net-(J4-Pad4) -> GBE0_MDI1+
- J4 pad 5: Net-(J4-Pad5) -> GBE0_MDI1-
- J4 pad 6: Net-(J4-Pad6) -> GBE0_CTREF(GND)
- J4 pad 7: Net-(J4-Pad7) -> GBE0_MDI2+
- J4 pad 8: Net-(J4-Pad8) -> GBE0_MDI2-
- J4 pad 9: Net-(J4-Pad9) -> GBE0_MDI3+
- J6 pad 1: mCOM_GND -> Net-(J6-Pad1)
- J7 pad 1: mCOM_GND -> GBE0_CTREF(GND)
- J8 pad 6: mCOM_GND -> GBE0_CTREF(GND)
- J9 pad 1: Net-(J9-Pad1) -> GPI0
- J9 pad 2: Net-(J9-Pad2) -> GPO0
- J9 pad 3: Net-(J9-Pad3) -> GPI1
- J9 pad 4: Net-(J9-Pad4) -> GPO1
- J9 pad 5: Net-(J9-Pad5) -> GPI2
- J9 pad 6: Net-(J9-Pad6) -> GPO2
- J9 pad 7: Net-(J9-Pad7) -> GPI3
- J9 pad 8: Net-(J9-Pad8) -> GPO3
- R23 pad 1: mCOM_GND -> GBE0_CTREF(GND)
- R24 pad 1: mCOM_GND -> GBE0_CTREF(GND)
- R25 pad 1: mCOM_GND -> GBE0_CTREF(GND)
- R3 pad 1: +12V -> mCOM_12V
- R32 pad 2: mCOM_GND -> GBE0_CTREF(GND)
- R7 pad 1: +12V -> mCOM_12V
- U1 pad 12: mCOM_GND -> GBE0_CTREF(GND)
- U1 pad 13: mCOM_GND -> GBE0_CTREF(GND)
- U1 pad 14: mCOM_GND -> GBE0_CTREF(GND)
- U1 pad 16: +12V -> mCOM_12V
- U2 pad 12: mCOM_GND -> GBE0_CTREF(GND)
- U2 pad 13: mCOM_GND -> GBE0_CTREF(GND)
- U2 pad 14: mCOM_GND -> GBE0_CTREF(GND)
- U2 pad 16: +12V -> mCOM_12V
- U9 pad 15: mCOM_GND -> GBE0_CTREF(GND)
- U9 pad 18: mCOM_GND -> GBE0_CTREF(GND)
- U9 pad 21: mCOM_GND -> GBE0_CTREF(GND)
- U9 pad 26: mCOM_GND -> GBE0_CTREF(GND)
- U9 pad 27: mCOM_GND -> GBE0_CTREF(GND)
- U9 pad 29: mCOM_GND -> GBE0_CTREF(GND)
- U9 pad 34: mCOM_GND -> GBE0_CTREF(GND)
- U9 pad 35: mCOM_GND -> GBE0_CTREF(GND)
- U9 pad 37: mCOM_GND -> GBE0_CTREF(GND)
- U9 pad 4: mCOM_GND -> GBE0_CTREF(GND)
- U9 pad 40: mCOM_GND -> GBE0_CTREF(GND)
- U9 pad 50: mCOM_GND -> GBE0_CTREF(GND)
- U9 pad 9: mCOM_GND -> GBE0_CTREF(GND)
