File: Carrier-Board.sch (KiCad schematic (older format))
At the start: 1 part, among them X1 PC104_PLUS

Commit message: Remove junk from pc104
Parts:
- removed X1: PC104_PLUS, Carrier-Board:con-pc104-PC104-PLUS, symbol PC104_PLUS
- added J1: PC104_PLUS, Carrier-Board:pc104_silk, symbol PC104_PLUS
Changed lines of the file:
@@
 EESchema Schematic File Version 2
+LIBS:Carrier-Board-rescue
 LIBS:power
 LIBS:device
@@
 LIBS:valves
 LIBS:Carrier-Board
+LIBS:SI-51009-F
 LIBS:Carrier-Board-cache
 EELAYER 25 0
@@
 $EndDescr
 $Comp
-L PC104_PLUS X1
-U 1 1 5A31DAD4
-P 3450 3050
-F 0 "X1" H 2950 4690 45  0000 L BNN
-F 1 "PC104_PLUS" H 2950 1250 45  0000 L BNN
-F 2 "Carrier-Board:con-pc104-PC104-PLUS" H 3480 3200 20  0001 C CNN
-F 3 "" H 3450 3050 60  0001 C CNN
-	1    3450 3050
+L PC104_PLUS J1
+U 1 1 5A6BBA3A
+P 2650 2600
+F 0 "J1" H 2150 4240 45  0000 L BNN
+F 1 "PC104_PLUS" H 2150 800 45  0000 L BNN
+F 2 "Carrier-Board:pc104_silk" H 2680 2750 20  0001 C CNN
+F 3 "" H 2650 2600 60  0001 C CNN
+	1    2650 2600
 	1    0    0    -1
 $EndComp
 $Comp
-L PC104_PLUS X1
-U 2 1 5A31DB5C
-P 5700 3050
-F 0 "X1" H 5200 4690 45  0000 L BNN
-F 1 "PC104_PLUS" H 5200 1250 45  0000 L BNN
-F 2 "Carrier-Board:con-pc104-PC104-PLUS" H 5730 3200 20  0001 C CNN
-F 3 "" H 5700 3050 60  0001 C CNN
-	2    5700 3050
+L PC104_PLUS J1
+U 2 1 5A6BBAB1
+P 5350 2950
+F 0 "J1" H 4850 4590 45  0000 L BNN
+F 1 "PC104_PLUS" H 4850 1150 45  0000 L BNN
+F 2 "Carrier-Board:pc104_silk" H 5380 3100 20  0001 C CNN
+F 3 "" H 5350 2950 60  0001 C CNN
+	2    5350 2950
 	1    0    0    -1
 $EndComp
 $Comp
-L PC104_PLUS X1
-U 3 1 5A31DBBB
-P 7300 3100
-F 0 "X1" H 6800 4740 45  0000 L BNN
-F 1 "PC104_PLUS" H 6800 1300 45  0000 L BNN
-F 2 "Carrier-Board:con-pc104-PC104-PLUS" H 7330 3250 20  0001 C CNN
-F 3 "" H 7300 3100 60  0001 C CNN
-	3    7300 3100
+L PC104_PLUS J1
+U 3 1 5A6BBB22
+P 8100 2950
+F 0 "J1" H 7600 4590 45  0000 L BNN
+F 1 "PC104_PLUS" H 7600 1150 45  0000 L BNN
+F 2 "Carrier-Board:pc104_silk" H 8130 3100 20  0001 C CNN
+F 3 "" H 8100 2950 60  0001 C CNN
+	3    8100 2950
 	1    0    0    -1
 $EndComp
 $Comp
-L PC104_PLUS X1
-U 4 1 5A31DC09
-P 8450 3050
-F 0 "X1" H 7950 4690 45  0000 L BNN
-F 1 "PC104_PLUS" H 7950 1250 45  0000 L BNN
-F 2 "Carrier-Board:con-pc104-PC104-PLUS" H 8480 3200 20  0001 C CNN
-F 3 "" H 8450 3050 60  0001 C CNN
-	4    8450 3050
+L PC104_PLUS J1
+U 4 1 5A6BBB83
+P 10050 2950
+F 0 "J1" H 9550 4590 45  0000 L BNN
+F 1 "PC104_PLUS" H 9550 1150 45  0000 L BNN
+F 2 "Carrier-Board:pc104_silk" H 10080 3100 20  0001 C CNN
+F 3 "" H 10050 2950 60  0001 C CNN
+	4    10050 2950
 	1    0    0    -1
 $EndComp
-$Comp
-L PC104_PLUS X1
-U 5 1 5A31DC65
-P 9900 3200
-F 0 "X1" H 9400 4840 45  0000 L BNN
-F 1 "PC104_PLUS" H 9400 1400 45  0000 L BNN
-F 2 "Carrier-Board:con-pc104-PC104-PLUS" H 9930 3350 20  0001 C CNN
-F 3 "" H 9900 3200 60  0001 C CNN
-	5    9900 3200
-	1    0    0    -1
-$EndComp
-$Comp
-L PC104_PLUS X1
-U 6 1 5A31DCC7
-P 10950 3200
-F 0 "X1" H 10450 4840 45  0000 L BNN
-F 1 "PC104_PLUS" H 10450 1400 45  0000 L BNN
-F 2 "Carrier-Board:con-pc104-PC104-PLUS" H 10980 3350 20  0001 C CNN
-F 3 "" H 10950 3200 60  0001 C CNN
-	6    10950 3200
-	1    0    0    -1
-$EndComp

Commit message: 'kidz
Parts:
- removed J1: PC104_PLUS, Carrier-Board:pc104_silk, symbol PC104_PLUS
- added J? (x2): Conn_02x26_Odd_Even, Carrier-Board:ESQ-126-XX-X-D, symbol Conn_02x26_Odd_Even
- added J?: SI-51009-F, Carrier-Board:SI-51009-F, symbol SI-51009-F
- added J? (x5): CONN_3-6318491-6, CONN_3-6318491-6, symbol CONN_3-6318491-6
- added U?: MSATA-Socket, Carrier-Board:msata-socket, symbol MSATA-Socket
Changed lines of the file:
@@
 $EndDescr
 $Comp
-L PC104_PLUS J1
-U 1 1 5A6BBA3A
-P 2650 2600
-F 0 "J1" H 2150 4240 45  0000 L BNN
-F 1 "PC104_PLUS" H 2150 800 45  0000 L BNN
-F 2 "Carrier-Board:pc104_silk" H 2680 2750 20  0001 C CNN
-F 3 "" H 2650 2600 60  0001 C CNN
-	1    2650 2600
+L Conn_02x26_Odd_Even J?
+U 1 1 5A6C2591
+P 3100 6250
+F 0 "J?" H 3150 7550 50  0000 C CNN
+F 1 "Conn_02x26_Odd_Even" H 3150 4850 50  0000 C CNN
+F 2 "Carrier-Board:ESQ-126-XX-X-D" H 3100 6250 50  0001 C CNN
+F 3 "" H 3100 6250 50  0001 C CNN
+	1    3100 6250
 	1    0    0    -1
 $EndComp
 $Comp
-L PC104_PLUS J1
-U 2 1 5A6BBAB1
-P 5350 2950
-F 0 "J1" H 4850 4590 45  0000 L BNN
-F 1 "PC104_PLUS" H 4850 1150 45  0000 L BNN
-F 2 "Carrier-Board:pc104_silk" H 5380 3100 20  0001 C CNN
-F 3 "" H 5350 2950 60  0001 C CNN
-	2    5350 2950
+L Conn_02x26_Odd_Even J?
+U 1 1 5A6C25B0
+P 3900 6200
+F 0 "J?" H 3950 7500 50  0000 C CNN
+F 1 "Conn_02x26_Odd_Even" H 3950 4800 50  0000 C CNN
+F 2 "Carrier-Board:ESQ-126-XX-X-D" H 3900 6200 50  0001 C CNN
+F 3 "" H 3900 6200 50  0001 C CNN
+	1    3900 6200
 	1    0    0    -1
 $EndComp
 $Comp
-L PC104_PLUS J1
-U 3 1 5A6BBB22
-P 8100 2950
-F 0 "J1" H 7600 4590 45  0000 L BNN
-F 1 "PC104_PLUS" H 7600 1150 45  0000 L BNN
-F 2 "Carrier-Board:pc104_silk" H 8130 3100 20  0001 C CNN
-F 3 "" H 8100 2950 60  0001 C CNN
-	3    8100 2950
+L SI-51009-F J?
+U 1 1 5A6C2649
+P 7050 5600
+F 0 "J?" H 7450 5750 50  0000 C CNN
+F 1 "SI-51009-F" H 7450 5050 50  0000 C CNN
+F 2 "Carrier-Board:SI-51009-F" H 7450 4950 50  0001 C CNN
+F 3 "http://belfuse.com/pdfs/SI-51009-F.pdf" H 7450 4850 50  0001 C CNN
+F 4 "Modular Connectors / Ethernet Connectors RJ45 Connector, 8 Position, 1 port" H 7450 4750 50  0001 C CNN "Description"
+F 5 "RS" H 7450 4650 50  0001 C CNN "Supplier_Name"
+F 6 "Bel-Stewart" H 7450 4450 50  0001 C CNN "Manufacturer_Name"
+F 7 "SI-51009-F" H 7450 4350 50  0001 C CNN "Manufacturer_Part_Number"
+	1    7050 5600
 	1    0    0    -1
 $EndComp
 $Comp
-L PC104_PLUS J1
-U 4 1 5A6BBB83
-P 10050 2950
-F 0 "J1" H 9550 4590 45  0000 L BNN
-F 1 "PC104_PLUS" H 9550 1150 45  0000 L BNN
-F 2 "Carrier-Board:pc104_silk" H 10080 3100 20  0001 C CNN
-F 3 "" H 10050 2950 60  0001 C CNN
-	4    10050 2950
+L MSATA-Socket U?
+U 1 1 5A6C270C
+P 11150 4900
+F 0 "U?" H 10750 6200 60  0000 C CNN
+F 1 "MSATA-Socket" H 11250 3350 60  0000 C CNN
+F 2 "Carrier-Board:msata-socket" H 11250 3900 60  0000 C CNN
+F 3 "" H 11250 3900 60  0000 C CNN
+	1    11150 4900
 	1    0    0    -1
 $EndComp
+$Comp
+L CONN_3-6318491-6 J?
+U 1 1 5A6C27F3
+P -1650 -3200
+F 0 "J?" H -1300 -2950 60  0000 C CNN
+F 1 "CONN_3-6318491-6" H -1250 -5400 60  0000 C CNN
+F 2 "CONN_3-6318491-6" H -1250 -5460 60  0001 C CNN
+F 3 "" H -1650 -3200 60  0000 C CNN
+	1    -1650 -3200
+	1    0    0    -1
+$EndComp
+$Comp
+L CONN_3-6318491-6 J?
+U 2 1 5A6C2830
+P -350 -3250
+F 0 "J?" H 0   -3000 60  0000 C CNN
+F 1 "CONN_3-6318491-6" H 50  -5450 60  0000 C CNN
+F 2 "CONN_3-6318491-6" H 50  -5510 60  0001 C CNN
+F 3 "" H -350 -3250 60  0000 C CNN
+	2    -350 -3250
+	1    0    0    -1
+$EndComp
+$Comp
+L CONN_3-6318491-6 J?
+U 3 1 5A6C2857
+P 950 -3250
+F 0 "J?" H 1300 -3000 60  0000 C CNN
+F 1 "CONN_3-6318491-6" H 1350 -5450 60  0000 C CNN
+F 2 "CONN_3-6318491-6" H 1350 -5510 60  0001 C CNN
+F 3 "" H 950 -3250 60  0000 C CNN
+	3    950  -3250
+	1    0    0    -1
+$EndComp
+$Comp
+L CONN_3-6318491-6 J?
+U 4 1 5A6C288E
+P 2050 -3400
+F 0 "J?" H 2400 -3150 60  0000 C CNN
+F 1 "CONN_3-6318491-6" H 2450 -5600 60  0000 C CNN
+F 2 "CONN_3-6318491-6" H 2450 -5660 60  0001 C CNN
+F 3 "" H 2050 -3400 60  0000 C CNN
+	4    2050 -3400
+	1    0    0    -1
+$EndComp
+$Comp
+L CONN_3-6318491-6 J?
+U 5 1 5A6C28CD
+P 3300 -3350
+F 0 "J?" H 3650 -3100 60  0000 C CNN
+F 1 "CONN_3-6318491-6" H 3700 -5550 60  0000 C CNN
+F 2 "CONN_3-6318491-6" H 3700 -5610 60  0001 C CNN
+F 3 "" H 3300 -3350 60  0000 C CNN
+	5    3300 -3350
+	1    0    0    -1
+$EndComp

Commit message: Add old schematic
Parts:
- added C1, C3: 10uF, BusSimulator:C22, symbol CP
- added C19, C20, C21, C27, C28, C29: .1uF, Capacitors_SMD:C_0603, symbol CP
- added C2, C4: 22uF, BusSimulator:C22, symbol CP
- added D5: D_Zener 9V, Diodes_SMD:D_SOD-323, symbol D_Zener
- added D6, D7, D8: LED, Diodes_SMD:D_1206, symbol LED
- added G1: LOGO, BusSimulator:LetSatLogo440, symbol LOGO
- added IC1, IC2, IC3: CS30CL, BusSimulator:SOT95P280X145-5N, symbol CS30CL
- added J1: CONN_3-6318491-6, BusSimulator:ComExpressMini10, symbol CONN_3-6318491-6
- added J2: OSTTA024163, BusSimulator:OSTTA024163, symbol OSTTA024163
- added J6: Conn_01x03, Pin_Headers:Pin_Header_Straight_1x03_Pitch2.54mm, symbol Conn_01x03
- added R1, R5: 160k, Resistors_SMD:R_0805, symbol R
- added R10, R12, R9: 10k, Resistors_SMD:R_0603, symbol R
- added R11: 30k, Resistors_SMD:R_0603, symbol R
- added R16, R17, R20: 25m, Resistors_SMD:R_0805, symbol R
- added R2: 30.1k, Resistors_SMD:R_0805, symbol R
- added R23: 330, Resistors_SMD:R_0603, symbol R
- added R24: 180, Resistors_SMD:R_0603, symbol R
- added R25: 1k, Resistors_SMD:R_0603, symbol R
- added R3, R7: 100k, Resistors_SMD:R_0805, symbol R
- added R32: 0, Resistors_SMD:R_0805, symbol R
- added R4: 63.4k, Resistors_SMD:R_0805, symbol R
- added R6: 51k, Resistors_SMD:R_0805, symbol R
- added R8: 56k, Resistors_SMD:R_0805, symbol R
- added U1, U2: MPM3620, BusSimulator:QFN-20, symbol MPM3620
- added U9: MSATA-Socket, BusSimulator:msata-socket, symbol MSATA-Socket
Connections:
- net labels added: +12V, +2.5V, +3.3V, +3V, +5V, 12v_sense, 3v3_sense, 5v_sense, Current_12v, Current_3v3, Current_5v, GNDA, GNDREF, GPI0, GPI1, GPI2, GPI3, GPO0, GPO1, GPO2, GPO3, I2C_CK, I2C_DAT, Load_1_PWR, Load_2_PWR, Load_3_PWR, PCE3895CT-ND, PCE3900CT-ND, PWRBTNn, PWR_OK, SATA0_RX+, SATA0_RX-, SATA0_TX+, SATA0_TX-, SATA_ACTn, SLEEPn, SYS_RESETn, WAKE1n, mCOM_12V, mCOM_5V_SBY, mCOM_GND, mCOM_RX, mCOM_TX, mCom_12V
- wire segments 0 -> 110
Other:
- note added: "1"
- note added: "12V\n"
- note added: "3V3\n"
- note added: "5V SBY\n"
- note added: "ADC\n"
- note added: "Amplifiers\n"
- note added: "Break out\n"
- note added: "Connectors\n"
- note added: "Current Sense\n"
- note added: "FALL 2017\n"
- note added: "Isolation\n\n"
- note added: "LED Indicators\n"
- note added: "LetSat-1 Bus Simulator"
- note added: "Microcontroller\n"
- note added: "Sata Connector\n"
- note added: "Voltage Supply"

Commit message: added footprints
Parts:
- removed C19, C20, C21: .1uF, Capacitors_SMD:C_0603, symbol CP
- removed IC1, IC2, IC3: CS30CL, BusSimulator:SOT95P280X145-5N, symbol CS30CL
- removed J2: OSTTA024163, BusSimulator:OSTTA024163, symbol OSTTA024163
- removed J6: Conn_01x03, Pin_Headers:Pin_Header_Straight_1x03_Pitch2.54mm, symbol Conn_01x03
- removed J? (x5): CONN_3-6318491-6, CONN_3-6318491-6, symbol CONN_3-6318491-6
- removed R16, R17, R20: 25m, Resistors_SMD:R_0805, symbol R
- removed U?: MSATA-Socket, Carrier-Board:msata-socket, symbol MSATA-Socket
- added J2: Conn_01x0, symbol Conn_01x03
- added J?: Conn_01x06_Male, symbol Conn_01x06_Male
- added J? (x2): Conn_01x03_Male, symbol Conn_01x03_Male
- gave numbers to parts that had none: 3
Connections:
- net labels removed: 3v3_sense, 5v_sense, Current_12v, Current_3v3, Current_5v, Load_1_PWR, Load_2_PWR, Load_3_PWR
- wire segments 110 -> 108
Other:
- note added: "LetSat-1 Carrier Prototype\n"
- note added: "Spring 2018\n\n"
- note removed: "ADC\n"
- note removed: "Amplifiers\n"
- note removed: "Connectors\n"
- note removed: "Current Sense\n"
- note removed: "FALL 2017\n"
- note removed: "Isolation\n\n"
- note removed: "LetSat-1 Bus Simulator"
- note removed: "Microcontroller\n"
- moved on the sheet: C1, C2, C27, C28, C29, C3, C4, D5, D6, D7, D8, J1A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

Commit message: schematic 90% done
Parts:
- removed R11: 30k, Resistors_SMD:R_0603, symbol R
- removed R12: 10k, Resistors_SMD:R_0603, symbol R
- added J9: Conn_02x04_Odd_Even, Pin_Headers:Pin_Header_Angled_2x04_Pitch2.54mm, symbol Conn_02x04_Odd_Even
- J6, J7: renamed from J?; footprint (none) -> Pin_Headers:Pin_Header_Angled_1x03_Pitch2.54mm
- J8: renamed from J?; footprint (none) -> Pin_Headers:Pin_Header_Angled_1x06_Pitch2.54mm
Connections:
- net +12V: now also C1.1, C3.2
- net +3V3: now also C4.1
- net +5V: now also C2.1
- net GNDREF: now also C1.2, C2.2, C3.1, C4.2
Other:
- moved on the sheet: C1, C2, C27, C28, C29, C3, C4, J6, J7, J8, R32, U9

Commit message: began layot
added dc jack, fixed ethernet footptrint aligned pc104
Parts:
- J2: footprint (none) -> Connectors:Barrel_Jack_CUI_PJ-036AH-SMT; symbol Conn_01x03 -> Barrel_Jack
- U9: footprint BusSimulator:msata-socket -> Carrier-Board:mpcie-socket
Connections:
- net +12V: now also J2.1; no longer J2.3 (Pin_3)
- net GNDREF: now also J2.3

Commit message: Finished Schmatic
Didnt do pc104 connector
Parts:
- removed R10, R9: 10k, Resistors_SMD:R_0603, symbol R
- added R?: 330, Resistors_SMD:R_0805, symbol R
- added R?: 330, symbol R
- J4: symbol SI-51009-F -> Conn_02x09_Odd_Even
Connections:
- net +12V: now also C3.1; no longer C3.2
- net GNDREF: now also C3.2, J1.14, J4.1 (Pin_1), J4.17 (Pin_17), J4.18 (Pin_18), J4.6 (Pin_6), R?.1, R?.1; no longer C3.1
- net GBE0_MDI1+: now reaches J1.10
- net GBE0_MDI1+: now also J4.4 (Pin_4)
- net GBE0_MDI0-: now reaches J1.12
- net GBE0_MDI0-: now also J4.3 (Pin_3)
- net GBE0_MDI0+: now reaches J1.13
- net GBE0_MDI0+: now also J4.2 (Pin_2)
- net GBE0_MDI3-: now reaches J1.2
- net GBE0_MDI3-: now also J4.10 (Pin_10)
- net GBE0_MDI3+: now reaches J1.3
- net GBE0_MDI3+: now also J4.9 (Pin_9)
- net GBE0_LINK100#: now reaches J1.4
- net GBE0_LINK100#: now also J4.16 (Pin_16)
- net GBE0_LINK1000#: now reaches J1.5
- net GBE0_LINK1000#: now also J4.13 (Pin_13)
- net GBE0_MDI2-: now reaches J1.6
- net GBE0_MDI2-: now also J4.8 (Pin_8)
- net GBE0_MDI2+: now reaches J1.7
- net GBE0_MDI2+: now also J4.7 (Pin_7)
- net GBE0_MDI1-: now reaches J1.9
- net GBE0_MDI1-: now also J4.5 (Pin_5)
- new net: J4.14 (Pin_14), R?.2
- new net: J4.15 (Pin_15), R?.2
Other:
- note added: "Ethernet"
- note added: "mCOMTK1\n"
- moved on the sheet: C1, C2, C27, C28, C29, C3, C4, D5, D6, D7, D8, J1A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

Commit message: Added SPI
Added SPI
Added GPIO
Fixed 12V
Parts:
- added J?: Conn_02x03_Odd_Even, symbol Conn_02x03_Odd_Even
Connections:
- net mCOM_12V is gone; now on net +12V: D5.1 (K), J1.104, J1.105, J1.106, J1.107, J1.108, J1.109, J1.214, J1.215, J1.216, J1.217, J1.218, J1.219
- net GNDREF: now also J?.6 (Pin_6); no longer J6.1 (Pin_1)
- net GPI0: now also J9.1 (Pin_1)
- net GPI1: now also J9.3 (Pin_3)
- net GPI2: now also J9.5 (Pin_5)
- net GPI3: now also J9.7 (Pin_7)
- net GPO0: now also J9.2 (Pin_2)
- net GPO1: now also J9.4 (Pin_4)
- net GPO2: now also J9.6 (Pin_6)
- net GPO3: now also J9.8 (Pin_8)
- net SPI_MISO: now reaches J1.92
- net SPI_MISO: now also J?.1 (Pin_1)
- net SPI_CLK: now reaches J1.94
- net SPI_CLK: now also J?.3 (Pin_3)
- net SPI_MOSI: now reaches J1.95
- net SPI_MOSI: now also J?.4 (Pin_4)
- net SPI_CS#: now reaches J1.97
- net SPI_CS#: now also J?.5 (Pin_5)
- new net SPI_POWER: J?.2 (Pin_2)
Other:
- note added: "GPIO\n"
- note added: "I2C\n"
- note added: "MISC SHIT"
- note added: "PC104\n"
- note added: "Rs232\n"
- note added: "SPI\n"
- moved on the sheet: J2, J8, J9
Changed lines of the file:
@@
 L +12V #PWR019
 U 1 1 5A0413FE
-P 1700 1950
-F 0 "#PWR019" H 1700 1800 50  0001 C CNN
-F 1 "+12V" H 1700 2090 50  0000 C CNN
-F 2 "" H 1700 1950 50  0001 C CNN
-F 3 "" H 1700 1950 50  0001 C CNN
-	1    1700 1950
+P 1250 1850
+F 0 "#PWR019" H 1250 1700 50  0001 C CNN
+F 1 "+12V" H 1250 1990 50  0000 C CNN
+F 2 "" H 1250 1850 50  0001 C CNN
+F 3 "" H 1250 1850 50  0001 C CNN
+	1    1250 1850
 	1    0    0    -1
 $EndComp
@@
 L GNDREF #PWR020
 U 1 1 5A04143A
-P 1350 1850
-F 0 "#PWR020" H 1350 1600 50  0001 C CNN
-F 1 "GNDREF" H 1350 1700 50  0000 C CNN
-F 2 "" H 1350 1850 50  0001 C CNN
-F 3 "" H 1350 1850 50  0001 C CNN
-	1    1350 1850
+P 900 1750
+F 0 "#PWR020" H 900 1500 50  0001 C CNN
+F 1 "GNDREF" H 900 1600 50  0000 C CNN
+F 2 "" H 900 1750 50  0001 C CNN
+F 3 "" H 900 1750 50  0001 C CNN
+	1    900  1750
 	1    0    0    -1
 $EndComp
@@
 Text GLabel 8750 1500 0    51   Input ~ 0
 I2C_DAT
-Text Notes 8300 1100 0    118  ~ 0
+Text Notes 8450 1050 0    118  ~ 0
 Break out\n
 $Comp
@@
 L GNDREF #PWR036
 U 1 1 5A0B68CF
-P 8750 1600
-F 0 "#PWR036" H 8750 1350 50  0001 C CNN
-F 1 "GNDREF" H 8750 1450 50  0000 C CNN
-F 2 "" H 8750 1600 50  0001 C CNN
-F 3 "" H 8750 1600 50  0001 C CNN
-	1    8750 1600
+P 8850 1600
+F 0 "#PWR036" H 8850 1350 50  0001 C CNN
+F 1 "GNDREF" H 8850 1450 50  0000 C CNN
+F 2 "" H 8850 1600 50  0001 C CNN
+F 3 "" H 8850 1600 50  0001 C CNN
+	1    8850 1600
 	1    0    0    -1
 $EndComp
@@
 L Barrel_Jack J2
 U 1 1 5A6C7CD3
-P 1450 1450
-F 0 "J2" H 1450 1550 50  0000 C CNN
-F 1 "Conn_01x0" H 1450 1250 50  0000 C CNN
-F 2 "Connectors:Barrel_Jack_CUI_PJ-036AH-SMT" H 1450 1450 50  0001 C CNN
-F 3 "" H 1450 1450 50  0001 C CNN
-	1    1450 1450
+P 1000 1350
+F 0 "J2" H 1000 1450 50  0000 C CNN
+F 1 "Conn_01x0" H 1000 1150 50  0000 C CNN
+F 2 "Connectors:Barrel_Jack_CUI_PJ-036AH-SMT" H 1000 1350 50  0001 C CNN
+F 3 "" H 1000 1350 50  0001 C CNN
+	1    1000 1350
 	0    1    1    0
 $EndComp
 Wire Wire Line
-	1550 1750 1550 2050
-Wire Wire Line
-	1550 2050 1700 2050
-Wire Wire Line
-	1700 2050 1700 1950
+	1100 1650 1100 1950
+Wire Wire Line
+	1100 1950 1250 1950
+Wire Wire Line
+	1250 1950 1250 1850
 Text GLabel 9800 1400 0    51   Input ~ 0
 mCOM_TX
@@
 L Conn_01x06_Male J8
 U 1 1 5A6CEF71
-P 10150 2350
-F 0 "J8" H 10150 2650 50  0000 C CNN
-F 1 "Conn_01x06_Male" H 10150 1950 50  0000 C CNN
-F 2 "Pin_Headers:Pin_Header_Angled_1x06_Pitch2.54mm" H 10150 2350 50  0001 C CNN
-F 3 "" H 10150 2350 50  0001 C CNN
-	1    10150 2350
+P 10450 2400
+F 0 "J8" H 10450 2700 50  0000 C CNN
+F 1 "Conn_01x06_Male" H 10450 2000 50  0000 C CNN
+F 2 "Pin_Headers:Pin_Header_Angled_1x06_Pitch2.54mm" H 10450 2400 50  0001 C CNN
+F 3 "" H 10450 2400 50  0001 C CNN
+	1    10450 2400
 	-1   0    0    1
 $EndComp
@@
 	-1   0    0    1
 $EndComp
-Text GLabel 9950 2050 0    51   Input ~ 0
+Text GLabel 10250 2100 0    51   Input ~ 0
 mCOM_GND
-Text GLabel 9950 2150 0    51   Input ~ 0
+Text GLabel 10250 2200 0    51   Input ~ 0
 PWRBTNn
-Text GLabel 9950 2250 0    51   Input ~ 0
+Text GLabel 10250 2300 0    51   Input ~ 0
 SYS_RESETn
-Text GLabel 9950 2350 0    51   Input ~ 0
+Text GLabel 10250 2400 0    51   Input ~ 0
 WAKE1n
-Text GLabel 9950 2450 0    51   Input ~ 0
+Text GLabel 10250 2500 0    51   Input ~ 0
 PWR_OK
-Text GLabel 9950 2550 0    51   Input ~ 0
+Text GLabel 10250 2600 0    51   Input ~ 0
 SLEEPn
 $Comp
 L Conn_02x04_Odd_Even J9
 U 1 1 5A6D35A7
-P 8800 2100
-F 0 "J9" H 8850 2300 50  0000 C CNN
-F 1 "Conn_02x04_Odd_Even" H 8850 1800 50  0000 C CNN
-F 2 "Pin_Headers:Pin_Header_Angled_2x04_Pitch2.54mm" H 8800 2100 50  0001 C CNN
-F 3 "" H 8800 2100 50  0001 C CNN
-	1    8800 2100
+P 8900 2100
+F 0 "J9" H 8950 2300 50  0000 C CNN
+F 1 "Conn_02x04_Odd_Even" H 8950 1800 50  0000 C CNN
+F 2 "Pin_Headers:Pin_Header_Angled_2x04_Pitch2.54mm" H 8900 2100 50  0001 C CNN
+F 3 "" H 8900 2100 50  0001 C CNN
+	1    8900 2100
 	1    0    0    -1
 $EndComp
 Connection ~ 2950 6250
 Wire Wire Line
-	1350 1750 1350 1850
-Wire Wire Line
-	1450 1750 1350 1750
+	900  1650 900  1750
+Wire Wire Line
+	1000 1650 900  1650
 Text GLabel 9450 4950 0    51   Input ~ 0
 GBE0_MDI3-
@@
 Text Notes 8550 4050 0    60   ~ 0
 mCOMTK1\n
+Text GLabel 1400 1850 2    51   Input ~ 0
+mCOM_12V
+Wire Wire Line
+	1250 1850 1400 1850
+Text GLabel 8700 2000 0    51   Input ~ 0
+GPI0
+Text GLabel 8700 2100 0    51   Input ~ 0
+GPI1
+Text GLabel 8700 2200 0    51   Input ~ 0
+GPI2
+Text GLabel 8700 2300 0    51   Input ~ 0
+GPI3
+Text GLabel 9200 2000 2    51   Input ~ 0
+GPO0
+Text GLabel 9200 2100 2    51   Input ~ 0
+GPO1
+Text GLabel 9200 2200 2    51   Input ~ 0
+GPO2
+Text GLabel 9200 2300 2    51   Input ~ 0
+GPO3
+$Comp
+L Conn_02x03_Odd_Even J?
+U 1 1 5A6E3060
+P 9100 2950
+F 0 "J?" H 9150 3150 50  0000 C CNN
+F 1 "Conn_02x03_Odd_Even" H 9150 2750 50  0000 C CNN
+F 2 "" H 9100 2950 50  0001 C CNN
+F 3 "" H 9100 2950 50  0001 C CNN
+	1    9100 2950
+	1    0    0    -1
+$EndComp
+Text GLabel 8900 3050 0    60   Input ~ 0
+SPI_CS#
+Text GLabel 8900 2850 0    60   Input ~ 0
+SPI_MISO
+Text GLabel 9400 2950 2    60   Input ~ 0
+SPI_MOSI
+Text GLabel 8900 2950 0    60   Input ~ 0
+SPI_CLK
+Text GLabel 9400 2850 2    60   Input ~ 0
+SPI_POWER
+Text GLabel 9400 3050 2    51   Input ~ 0
+mCOM_GND
+Text GLabel 12450 5650 0    60   Input ~ 0
+SPI_CS#
+Text GLabel 12450 5150 0    60   Input ~ 0
+SPI_MISO
+Text GLabel 12450 5350 0    60   Input ~ 0
+SPI_CLK
+Text GLabel 12450 5450 0    60   Input ~ 0
+SPI_MOSI
+Text Notes 8450 1250 0    60   ~ 0
+I2C\n
+Text Notes 9600 1250 0    60   ~ 0
+Rs232\n
+Text Notes 8500 2750 0    60   ~ 0
+SPI\n
+Text Notes 8450 1900 0    60   ~ 0
+GPIO\n
+Text Notes 9850 1950 0    60   ~ 0
+MISC SHIT
+Text Notes 11600 700  0    60   ~ 0
+PC104\n
 $EndSCHEMATC
